Commit message: increase effort of the grippers

File: src/curobo/content/assets/robot/franka_description/dual_panda_shoulder.urdf (robot description, URDF)
Before this commit: robot dual_panda, 29 links, 28 joints
Joints:
- joint panda1_finger_joint1: limit lower=0.0 upper=0.04 effort=20 velocity=0.2 -> lower=0.0 upper=0.04 effort=200 velocity=0.2
- joint panda1_finger_joint2: limit lower=0.0 upper=0.04 effort=20 velocity=0.2 -> lower=0.0 upper=0.04 effort=200 velocity=0.2
- joint panda2_finger_joint1: limit lower=0.0 upper=0.04 effort=20 velocity=0.2 -> lower=0.0 upper=0.04 effort=200 velocity=0.2
- joint panda2_finger_joint2: limit lower=0.0 upper=0.04 effort=20 velocity=0.2 -> lower=0.0 upper=0.04 effort=200 velocity=0.2
